Commit message: Change phantomx mass and color

File: urdf/phantomx_urdf.xacro (robot description, xacro)
@@ -121,5 +121,5 @@
     </inertial>
     <visual>
-      <origin xyz="0 0 0" rpy="0 0 0"  />
+      <origin xyz="0 0 0" rpy="-5 0 0"  />
       <geometry>
         <!--box size="0.045 0.022 0.0325" /-->
@@ -131,5 +131,5 @@
     </visual>
     <collision>
-      <origin xyz="0 0 0" rpy="0 0 0"  />
+      <origin xyz="0 0 0" rpy="-5 0 0"  />
       <geometry>
         <mesh filename="package://phantomx_description/meshes/tibia_l_coll.STL"  scale="1 1 1"/>
