Commit message: Change mass and color.

File: urdf/phantomx.urdf (robot description, URDF)
Before this commit: robot PhantomX, 26 links, 25 joints
Links:
- link MP_BODY: mass 0.97559947 -> 2.27559947
- link c1_lf: mass 0.024357719 -> 0.524357719
- link c1_lm: mass 0.024357719 -> 0.524357719
- link c1_lr: mass 0.024357719 -> 0.524357719
- link c1_rf: mass 0.024357719 -> 0.524357719
- link c1_rm: mass 0.024357719 -> 0.524357719
- link c1_rr: mass 0.024357719 -> 0.524357719
- link c2_lf: mass 0.024357719 -> 0.524357719
- link c2_lm: mass 0.024357719 -> 0.524357719
- link c2_lr: mass 0.024357719 -> 0.524357719
- link c2_rf: mass 0.024357719 -> 0.524357719
- link c2_rm: mass 0.024357719 -> 0.524357719
- link c2_rr: mass 0.024357719 -> 0.524357719
- link thigh_lf: mass 0.024357719 -> 0.524357719
- link thigh_lm: mass 0.024357719 -> 0.524357719
- link thigh_lr: mass 0.024357719 -> 0.524357719
- link thigh_rf: mass 0.024357719 -> 0.524357719
- link thigh_rm: mass 0.024357719 -> 0.524357719
- link thigh_rr: mass 0.024357719 -> 0.524357719
- link tibia_lf: mass 0.024357719 -> 0.524357719
- link tibia_lm: mass 0.024357719 -> 0.524357719
- link tibia_lr: mass 0.024357719 -> 0.524357719
- link tibia_rf: mass 0.024357719 -> 0.524357719
- link tibia_rm: mass 0.024357719 -> 0.524357719
- link tibia_rr: mass 0.024357719 -> 0.524357719
Joints:
- joint j_thigh_lf: origin xyz=0 0 0 rpy=3.14159 0  0 -> xyz=0 0 0 rpy= 0 3.14159 3.14159
- joint j_thigh_lm: origin xyz=0 0 0 rpy=3.14159 0  0 -> xyz=0 0 0 rpy= 0 3.14159 3.14159
- joint j_thigh_lr: origin xyz=0 0 0 rpy=3.14159 0  0 -> xyz=0 0 0 rpy= 0 3.14159 3.14159
- joint j_thigh_rf: origin xyz=0 0 0 rpy=3.14159 0  0 -> xyz=0 0 0 rpy= 0 3.14159 3.14159
- joint j_thigh_rm: origin xyz=0 0 0 rpy=3.14159 0  0 -> xyz=0 0 0 rpy= 0 3.14159 3.14159
- joint j_thigh_rr: origin xyz=0 0 0 rpy=3.14159 0  0 -> xyz=0 0 0 rpy= 0 3.14159 3.14159

File: urdf/phantomx_urdf.xacro (robot description, xacro)
@@ -8,10 +8,10 @@
         <parent link="${parent}"/>
         <child link="MP_BODY"/>
-        <insert_block name="origin" />
+        <xacro:insert_block name="origin" />
       </joint>
       <link name="MP_BODY">
         <inertial>
           <origin xyz="0 0 0" />
-          <mass value="0.97559947"/>
+          <mass value="2.27559947"/>
           <inertia ixx="3.1081800"  ixy="-0.25460189"  ixz="2.0318174" iyy="6.3787776" iyz="0.16417863" izz="5.3316425" />
         </inertial>
@@ -35,5 +35,5 @@
       </link>
       <gazebo reference="MP_BODY">
-        <material>Gazebo/Grey</material>
+        <material>Gazebo/Orange</material>
       </gazebo>
     <xacro:leg_l xyz="0.1248 -0.06164  0.001116"  rpy="0 4.7123 0.7853981633974483" suffix="rf"/>
@@ -48,5 +48,5 @@
     <inertial>
       <origin xyz="0 -${connect_offset} 0" rpy="0 0 0"  />
-      <mass value="0.024357719"/>
+      <mass value="0.524357719"/>
      <inertia ixx="0.0051411124"  ixy="-0.00057530255"  ixz="-0.000024729049" iyy="0.0081915737" iyz="-0.000019223094" izz="0.0011379812" />
     </inertial>
@@ -71,5 +71,5 @@
     <inertial>
       <origin xyz="0 -${connect_offset} 0" rpy="0 0 0"  />
-      <mass value="0.024357719"/>
+      <mass value="0.524357719"/>
      <inertia ixx="0.0051411124"  ixy="-0.00057530255"  ixz="-0.000024729049" iyy="0.0081915737" iyz="-0.000019223094" izz="0.0011379812" />
     </inertial>
@@ -94,5 +94,5 @@
     <inertial>
       <origin xyz="0 0 0" rpy="0 0 0"  />
-      <mass value="0.024357719"/>
+      <mass value="0.524357719"/>
      <inertia ixx="0.0051411124"  ixy="-0.00057530255"  ixz="-0.000024729049" iyy="0.0081915737" iyz="-0.000019223094" izz="0.0011379812" />
     </inertial>
@@ -117,5 +117,5 @@
     <inertial>
       <origin xyz="0 0 0" rpy="0 0 0"  />
-      <mass value="0.024357719"/>
+      <mass value="0.524357719"/>
      <inertia ixx="0.0051411124"  ixy="-0.00057530255"  ixz="-0.000024729049" iyy="0.0081915737" iyz="-0.000019223094" izz="0.0011379812" />
     </inertial>
@@ -135,6 +135,38 @@
         <mesh filename="package://phantomx_description/meshes/tibia_l_coll.STL"  scale="1 1 1"/>
       </geometry>
-    </collision>
-  </link>
+      <!--surface>
+          <friction>
+            <ode>
+              <mu>1000000.0</mu>
+              <mu2>1000000.0</mu2>
+              <slip1>0.0</slip1>
+              <slip2>0.0</slip2>
+            </ode>
+          </friction>
+        </surface-->
+    </collision>
+  </link>
+  <!--link name="contact_sensor_${suffix}">
+    <inertial>
+      <origin xyz="0 0 0" rpy="0 0 0" />
+      <mass value="0"/>
+     <inertia ixx="0.0"  ixy="0.0"  ixz="0.0" iyy="0.0" iyz="0.0" izz="0.0" />
+    </inertial>
+    <visual>
+      <origin xyz="0 0 0" rpy="0 0 0" />
+      <geometry>
+        <box size="0.005 0.011 0.005" />
+      </geometry>
+      <material name="Grey">
+        <color rgba="0.20 0.20 0.20 1.0"/>
+      </material>
+    </visual>
+    <collision name="collision_${suffix}">
+      <origin xyz="0 0 0" rpy="0 0 0" />
+      <geometry>
+        <box size="0.005 0.011 0.005" />
+      </geometry>
+    </collision>
+  </link-->
   <joint name="j_c1_${suffix}" type="revolute">
     <parent link="MP_BODY"/>
@@ -163,11 +195,16 @@
     <limit effort="2.8" velocity="5.6548668" lower="-2.6179939" upper="2.6179939" />
   </joint>
+  <!--joint name="j_contact_sensor_${suffix}" type="fixed">
+    <parent link="tibia_${suffix}"/>
+    <child link="contact_sensor_${suffix}"/>
+    <origin xyz="0.0017 0.1602 0.029" rpy="0 0 0" />
+  </joint-->
    <transmission name="t_c1_${suffix}">
     <type>transmission_interface/SimpleTransmission</type>
     <joint name="j_c1_${suffix}">
-      <hardwareInterface>EffortJointInterface</hardwareInterface>
+      <hardwareInterface>hardware_interface/EffortJointInterface</hardwareInterface>
     </joint>
     <actuator name="m_c1_${suffix}">
-      <hardwareInterface>EffortJointInterface</hardwareInterface>
+      <hardwareInterface>hardware_interface/EffortJointInterface</hardwareInterface>
       <mechanicalReduction>1</mechanicalReduction>
     </actuator>
@@ -176,8 +213,8 @@
     <type>transmission_interface/SimpleTransmission</type>
     <joint name="j_thigh_${suffix}">
-      <hardwareInterface>EffortJointInterface</hardwareInterface>
+      <hardwareInterface>hardware_interface/EffortJointInterface</hardwareInterface>
     </joint>
     <actuator name="m_thigh_${suffix}">
-      <hardwareInterface>EffortJointInterface</hardwareInterface>
+      <hardwareInterface>hardware_interface/EffortJointInterface</hardwareInterface>
       <mechanicalReduction>1</mechanicalReduction>
     </actuator>
@@ -186,8 +223,8 @@
     <type>transmission_interface/SimpleTransmission</type>
     <joint name="j_tibia_${suffix}">
-      <hardwareInterface>EffortJointInterface</hardwareInterface>
+      <hardwareInterface>hardware_interface/EffortJointInterface</hardwareInterface>
     </joint>
     <actuator name="m_tibia_${suffix}">
-      <hardwareInterface>EffortJointInterface</hardwareInterface>
+      <hardwareInterface>hardware_interface/EffortJointInterface</hardwareInterface>
       <mechanicalReduction>1</mechanicalReduction>
     </actuator>
@@ -197,5 +234,5 @@
   </gazebo>
   <gazebo reference="c2_${suffix}">
-    <material>Gazebo/Grey</material>
+    <material>Gazebo/Orange</material>
   </gazebo>
   <gazebo reference="thigh_${suffix}">
@@ -203,5 +240,5 @@
   </gazebo>
   <gazebo reference="tibia_${suffix}">
-    <material>Gazebo/Grey</material>
+    <material>Gazebo/Orange</material>
   </gazebo>
 </xacro:macro>

Commit message: Add dampening and collision to joints and links. Add new collision mesh for tibia

File: urdf/phantomx.urdf (robot description, URDF)
Before this commit: robot PhantomX, 26 links, 25 joints
Links:
- link MP_BODY: mass 2.27559947 -> 1.97559947
Joints:
- joint j_c1_lf: limit lower=-2.6179939 upper=2.6179939 effort=2.8 velocity=5.6548668 -> lower=-2.5179939 upper=2.5179939 effort=2.8 velocity=5.6548668
- joint j_c1_lm: limit lower=-2.6179939 upper=2.6179939 effort=2.8 velocity=5.6548668 -> lower=-2.5179939 upper=2.5179939 effort=2.8 velocity=5.6548668
- joint j_c1_lr: limit lower=-2.6179939 upper=2.6179939 effort=2.8 velocity=5.6548668 -> lower=-2.5179939 upper=2.5179939 effort=2.8 velocity=5.6548668
- joint j_c1_rf: limit lower=-2.6179939 upper=2.6179939 effort=2.8 velocity=5.6548668 -> lower=-2.5179939 upper=2.5179939 effort=2.8 velocity=5.6548668
- joint j_c1_rm: limit lower=-2.6179939 upper=2.6179939 effort=2.8 velocity=5.6548668 -> lower=-2.5179939 upper=2.5179939 effort=2.8 velocity=5.6548668
- joint j_c1_rr: limit lower=-2.6179939 upper=2.6179939 effort=2.8 velocity=5.6548668 -> lower=-2.5179939 upper=2.5179939 effort=2.8 velocity=5.6548668
- joint j_thigh_lf: limit lower=-2.6179939 upper=2.6179939 effort=2.8 velocity=5.6548668 -> lower=-2.5179939 upper=2.5179939 effort=2.8 velocity=5.6548668
- joint j_thigh_lm: limit lower=-2.6179939 upper=2.6179939 effort=2.8 velocity=5.6548668 -> lower=-2.5179939 upper=2.5179939 effort=2.8 velocity=5.6548668
- joint j_thigh_lr: limit lower=-2.6179939 upper=2.6179939 effort=2.8 velocity=5.6548668 -> lower=-2.5179939 upper=2.5179939 effort=2.8 velocity=5.6548668
- joint j_thigh_rf: limit lower=-2.6179939 upper=2.6179939 effort=2.8 velocity=5.6548668 -> lower=-2.5179939 upper=2.5179939 effort=2.8 velocity=5.6548668
- joint j_thigh_rm: limit lower=-2.6179939 upper=2.6179939 effort=2.8 velocity=5.6548668 -> lower=-2.5179939 upper=2.5179939 effort=2.8 velocity=5.6548668
- joint j_thigh_rr: limit lower=-2.6179939 upper=2.6179939 effort=2.8 velocity=5.6548668 -> lower=-2.5179939 upper=2.5179939 effort=2.8 velocity=5.6548668
- joint j_tibia_lf: limit lower=-2.6179939 upper=2.6179939 effort=2.8 velocity=5.6548668 -> lower=-2.6179939 upper=0.6179939 effort=2.8 velocity=5.6548668
- joint j_tibia_lm: limit lower=-2.6179939 upper=2.6179939 effort=2.8 velocity=5.6548668 -> lower=-2.6179939 upper=0.6179939 effort=2.8 velocity=5.6548668
- joint j_tibia_lr: limit lower=-2.6179939 upper=2.6179939 effort=2.8 velocity=5.6548668 -> lower=-2.6179939 upper=0.6179939 effort=2.8 velocity=5.6548668
- joint j_tibia_rf: limit lower=-2.6179939 upper=2.6179939 effort=2.8 velocity=5.6548668 -> lower=-2.6179939 upper=0.6179939 effort=2.8 velocity=5.6548668
- joint j_tibia_rm: limit lower=-2.6179939 upper=2.6179939 effort=2.8 velocity=5.6548668 -> lower=-2.6179939 upper=0.6179939 effort=2.8 velocity=5.6548668
- joint j_tibia_rr: limit lower=-2.6179939 upper=2.6179939 effort=2.8 velocity=5.6548668 -> lower=-2.6179939 upper=0.6179939 effort=2.8 velocity=5.6548668

File: urdf/phantomx_urdf.xacro (robot description, xacro)
@@ -10,8 +10,11 @@
         <xacro:insert_block name="origin" />
       </joint>
+      <gazebo reference="j_phantomx_attachment">
+        <implicitSpringDamper>1</implicitSpringDamper>
+      </gazebo>
       <link name="MP_BODY">
         <inertial>
           <origin xyz="0 0 0" />
-          <mass value="2.27559947"/>
+          <mass value="1.97559947"/>
           <inertia ixx="3.1081800"  ixy="-0.25460189"  ixz="2.0318174" iyy="6.3787776" iyz="0.16417863" izz="5.3316425" />
         </inertial>
@@ -36,4 +39,6 @@
       <gazebo reference="MP_BODY">
         <material>Gazebo/Orange</material>
+        <dampingFactor>.1</dampingFactor>
+        <selfCollide>1</selfCollide>
       </gazebo>
     <xacro:leg_l xyz="0.1248 -0.06164  0.001116"  rpy="0 4.7123 0.7853981633974483" suffix="rf"/>
@@ -52,5 +57,5 @@
     </inertial>
     <visual>
-      <origin xyz="0 -0.0252 0" rpy="0 0 0"  />
+      <origin xyz="0 -${connect_offset} 0" rpy="0 0 0"  />
       <geometry>
         <!--box size="0.045 0.022 0.0325" /-->
@@ -75,5 +80,5 @@
     </inertial>
     <visual>
-      <origin xyz="0 -0.0252 0" rpy="0 0 0"  />
+      <origin xyz="0 -${connect_offset} 0" rpy="0 0 0"  />
       <geometry>
         <!--box size="0.045 0.022 0.0325" /-->
@@ -116,12 +121,11 @@
   <link name="tibia_${suffix}">
     <inertial>
-      <origin xyz="0 0 0" rpy="0 0 0"  />
-      <mass value="0.524357719"/>
-     <inertia ixx="0.0051411124"  ixy="-0.00057530255"  ixz="-0.000024729049" iyy="0.0081915737" iyz="-0.000019223094" izz="0.0011379812" />
-    </inertial>
-    <visual>
       <origin xyz="0 0 0" rpy="-5 0 0"  />
-      <geometry>
-        <!--box size="0.045 0.022 0.0325" /-->
+      <mass value="0.524357719"/>
+     <inertia ixx="0.0051411124"  ixy="-0.00057530255"  ixz="-0.000024729049" iyy="0.0081915737" iyz="-0.000019223094" izz="0.0011379812" />
+    </inertial>
+    <visual>
+      <origin xyz="0 0 0" rpy="-5 0 0"  />
+      <geometry>
         <mesh filename="package://phantomx_description/meshes/tibia_l.STL"  scale="1 1 1"/>
       </geometry>
@@ -135,38 +139,6 @@
         <mesh filename="package://phantomx_description/meshes/tibia_l_coll.STL"  scale="1 1 1"/>
       </geometry>
-      <!--surface>
-          <friction>
-            <ode>
-              <mu>1000000.0</mu>
-              <mu2>1000000.0</mu2>
-              <slip1>0.0</slip1>
-              <slip2>0.0</slip2>
-            </ode>
-          </friction>
-        </surface-->
-    </collision>
-  </link>
-  <!--link name="contact_sensor_${suffix}">
-    <inertial>
-      <origin xyz="0 0 0" rpy="0 0 0" />
-      <mass value="0"/>
-     <inertia ixx="0.0"  ixy="0.0"  ixz="0.0" iyy="0.0" iyz="0.0" izz="0.0" />
-    </inertial>
-    <visual>
-      <origin xyz="0 0 0" rpy="0 0 0" />
-      <geometry>
-        <box size="0.005 0.011 0.005" />
-      </geometry>
-      <material name="Grey">
-        <color rgba="0.20 0.20 0.20 1.0"/>
-      </material>
-    </visual>
-    <collision name="collision_${suffix}">
-      <origin xyz="0 0 0" rpy="0 0 0" />
-      <geometry>
-        <box size="0.005 0.011 0.005" />
-      </geometry>
-    </collision>
-  </link-->
+    </collision>
+  </link>
   <joint name="j_c1_${suffix}" type="revolute">
     <parent link="MP_BODY"/>
@@ -174,5 +146,5 @@
     <origin xyz="${xyz}" rpy="${rpy}" />
     <axis xyz="1 0 0" />
-    <limit effort="2.8" velocity="5.6548668" lower="-2.6179939" upper="2.6179939" />
+    <limit effort="2.8" velocity="5.6548668" lower="-2.5179939" upper="2.5179939" />
   </joint>
   <joint name="j_c2_${suffix}" type="fixed">
@@ -186,5 +158,5 @@
     <origin xyz="0 0 0" rpy=" 0 3.14159 3.14159" />
     <axis xyz="1 0 0" />
-    <limit effort="2.8" velocity="5.6548668" lower="-2.6179939" upper="2.6179939" />
+    <limit effort="2.8" velocity="5.6548668" lower="-2.5179939" upper="2.5179939" />
   </joint>
   <joint name="j_tibia_${suffix}" type="revolute">
@@ -193,11 +165,6 @@
     <origin xyz="0 ${thigh_offset_y} ${thigh_offset_z}" rpy="-1.5707 0 3.14159" />
     <axis xyz="1 0 0" />
-    <limit effort="2.8" velocity="5.6548668" lower="-2.6179939" upper="2.6179939" />
-  </joint>
-  <!--joint name="j_contact_sensor_${suffix}" type="fixed">
-    <parent link="tibia_${suffix}"/>
-    <child link="contact_sensor_${suffix}"/>
-    <origin xyz="0.0017 0.1602 0.029" rpy="0 0 0" />
-  </joint-->
+    <limit effort="2.8" velocity="5.6548668" lower="-2.6179939" upper="0.6179939" />
+  </joint>
    <transmission name="t_c1_${suffix}">
     <type>transmission_interface/SimpleTransmission</type>
@@ -232,13 +199,30 @@
   <gazebo reference="c1_${suffix}">
     <material>Gazebo/Grey</material>
+        <dampingFactor>.1</dampingFactor>
   </gazebo>
   <gazebo reference="c2_${suffix}">
     <material>Gazebo/Orange</material>
+        <dampingFactor>.1</dampingFactor>
   </gazebo>
   <gazebo reference="thigh_${suffix}">
     <material>Gazebo/Grey</material>
+        <dampingFactor>.1</dampingFactor>
   </gazebo>
   <gazebo reference="tibia_${suffix}">
     <material>Gazebo/Orange</material>
+        <dampingFactor>.1</dampingFactor>
+        <selfCollide>1</selfCollide>
+  </gazebo>
+  <gazebo reference="j_c1_${suffix}">
+    <implicitSpringDamper>1</implicitSpringDamper>
+  </gazebo>
+  <gazebo reference="j_c2_${suffix}">
+    <implicitSpringDamper>1</implicitSpringDamper>
+  </gazebo>
+  <gazebo reference="j_thigh_${suffix}">
+    <implicitSpringDamper>1</implicitSpringDamper>
+  </gazebo>
+  <gazebo reference="j_tibia_${suffix}">
+    <implicitSpringDamper>1</implicitSpringDamper>
   </gazebo>
 </xacro:macro>

Commit message: Change Damping factor

File: urdf/phantomx.urdf (robot description, URDF)
Before this commit: robot PhantomX, 26 links, 25 joints
Links:
- link c1_lf: mass 0.524357719 -> 0.324357719
- link c1_lm: mass 0.524357719 -> 0.324357719
- link c1_lr: mass 0.524357719 -> 0.324357719
- link c1_rf: mass 0.524357719 -> 0.324357719
- link c1_rm: mass 0.524357719 -> 0.324357719
- link c1_rr: mass 0.524357719 -> 0.324357719
- link c2_lf: mass 0.524357719 -> 0.324357719
- link c2_lm: mass 0.524357719 -> 0.324357719
- link c2_lr: mass 0.524357719 -> 0.324357719
- link c2_rf: mass 0.524357719 -> 0.324357719
- link c2_rm: mass 0.524357719 -> 0.324357719
- link c2_rr: mass 0.524357719 -> 0.324357719
- link thigh_lf: mass 0.524357719 -> 0.324357719
- link thigh_lm: mass 0.524357719 -> 0.324357719
- link thigh_lr: mass 0.524357719 -> 0.324357719
- link thigh_rf: mass 0.524357719 -> 0.324357719
- link thigh_rm: mass 0.524357719 -> 0.324357719
- link thigh_rr: mass 0.524357719 -> 0.324357719
- link tibia_lf: mass 0.524357719 -> 0.324357719
- link tibia_lm: mass 0.524357719 -> 0.324357719
- link tibia_lr: mass 0.524357719 -> 0.324357719
- link tibia_rf: mass 0.524357719 -> 0.324357719
- link tibia_rm: mass 0.524357719 -> 0.324357719
- link tibia_rr: mass 0.524357719 -> 0.324357719

File: urdf/phantomx_urdf.xacro (robot description, xacro)
@@ -39,5 +39,5 @@
       <gazebo reference="MP_BODY">
         <material>Gazebo/Orange</material>
-        <dampingFactor>.1</dampingFactor>
+        <dampingFactor>0.001</dampingFactor>
         <selfCollide>1</selfCollide>
       </gazebo>
@@ -53,5 +53,5 @@
     <inertial>
       <origin xyz="0 -${connect_offset} 0" rpy="0 0 0"  />
-      <mass value="0.524357719"/>
+      <mass value="0.324357719"/>
      <inertia ixx="0.0051411124"  ixy="-0.00057530255"  ixz="-0.000024729049" iyy="0.0081915737" iyz="-0.000019223094" izz="0.0011379812" />
     </inertial>
@@ -76,5 +76,5 @@
     <inertial>
       <origin xyz="0 -${connect_offset} 0" rpy="0 0 0"  />
-      <mass value="0.524357719"/>
+      <mass value="0.324357719"/>
      <inertia ixx="0.0051411124"  ixy="-0.00057530255"  ixz="-0.000024729049" iyy="0.0081915737" iyz="-0.000019223094" izz="0.0011379812" />
     </inertial>
@@ -99,5 +99,5 @@
     <inertial>
       <origin xyz="0 0 0" rpy="0 0 0"  />
-      <mass value="0.524357719"/>
+      <mass value="0.324357719"/>
      <inertia ixx="0.0051411124"  ixy="-0.00057530255"  ixz="-0.000024729049" iyy="0.0081915737" iyz="-0.000019223094" izz="0.0011379812" />
     </inertial>
@@ -122,5 +122,5 @@
     <inertial>
       <origin xyz="0 0 0" rpy="-5 0 0"  />
-      <mass value="0.524357719"/>
+      <mass value="0.324357719"/>
      <inertia ixx="0.0051411124"  ixy="-0.00057530255"  ixz="-0.000024729049" iyy="0.0081915737" iyz="-0.000019223094" izz="0.0011379812" />
     </inertial>
@@ -199,17 +199,17 @@
   <gazebo reference="c1_${suffix}">
     <material>Gazebo/Grey</material>
-        <dampingFactor>.1</dampingFactor>
+        <dampingFactor>.001</dampingFactor>
   </gazebo>
   <gazebo reference="c2_${suffix}">
     <material>Gazebo/Orange</material>
-        <dampingFactor>.1</dampingFactor>
+        <dampingFactor>.01</dampingFactor>
   </gazebo>
   <gazebo reference="thigh_${suffix}">
     <material>Gazebo/Grey</material>
-        <dampingFactor>.1</dampingFactor>
+        <dampingFactor>.01</dampingFactor>
   </gazebo>
   <gazebo reference="tibia_${suffix}">
     <material>Gazebo/Orange</material>
-        <dampingFactor>.1</dampingFactor>
+        <dampingFactor>.01</dampingFactor>
         <selfCollide>1</selfCollide>
   </gazebo>
