Commit message: Change joint ranges

File: urdf/phantomx.urdf (robot description, URDF)
Before this commit: robot PhantomX, 26 links, 25 joints
Joints:
- joint j_c1_lf: limit lower=-2.5179939 upper=2.5179939 effort=2.8 velocity=5.6548668 -> lower=-0.523599 upper=0.523599 effort=2.8 velocity=5.6548668
- joint j_c1_lm: limit lower=-2.5179939 upper=2.5179939 effort=2.8 velocity=5.6548668 -> lower=-0.523599 upper=0.523599 effort=2.8 velocity=5.6548668
- joint j_c1_lr: limit lower=-2.5179939 upper=2.5179939 effort=2.8 velocity=5.6548668 -> lower=-0.523599 upper=0.523599 effort=2.8 velocity=5.6548668
- joint j_c1_rf: limit lower=-2.5179939 upper=2.5179939 effort=2.8 velocity=5.6548668 -> lower=-0.523599 upper=0.523599 effort=2.8 velocity=5.6548668
- joint j_c1_rm: limit lower=-2.5179939 upper=2.5179939 effort=2.8 velocity=5.6548668 -> lower=-0.523599 upper=0.523599 effort=2.8 velocity=5.6548668
- joint j_c1_rr: limit lower=-2.5179939 upper=2.5179939 effort=2.8 velocity=5.6548668 -> lower=-0.523599 upper=0.523599 effort=2.8 velocity=5.6548668
- joint j_thigh_lf: limit lower=-2.5179939 upper=2.5179939 effort=2.8 velocity=5.6548668 -> lower=-1.5708 upper=1.5708 effort=2.8 velocity=5.6548668
- joint j_thigh_lm: limit lower=-2.5179939 upper=2.5179939 effort=2.8 velocity=5.6548668 -> lower=-1.5708 upper=1.5708 effort=2.8 velocity=5.6548668
- joint j_thigh_lr: limit lower=-2.5179939 upper=2.5179939 effort=2.8 velocity=5.6548668 -> lower=-1.5708 upper=1.5708 effort=2.8 velocity=5.6548668
- joint j_thigh_rf: limit lower=-2.5179939 upper=2.5179939 effort=2.8 velocity=5.6548668 -> lower=-1.5708 upper=1.5708 effort=2.8 velocity=5.6548668
- joint j_thigh_rm: limit lower=-2.5179939 upper=2.5179939 effort=2.8 velocity=5.6548668 -> lower=-1.5708 upper=1.5708 effort=2.8 velocity=5.6548668
- joint j_thigh_rr: limit lower=-2.5179939 upper=2.5179939 effort=2.8 velocity=5.6548668 -> lower=-1.5708 upper=1.5708 effort=2.8 velocity=5.6548668
- joint j_tibia_lf: limit lower=-2.6179939 upper=0.6179939 effort=2.8 velocity=5.6548668 -> lower=-1.5708 upper=0.6179939 effort=2.8 velocity=5.6548668
- joint j_tibia_lm: limit lower=-2.6179939 upper=0.6179939 effort=2.8 velocity=5.6548668 -> lower=-1.5708 upper=0.6179939 effort=2.8 velocity=5.6548668
- joint j_tibia_lr: limit lower=-2.6179939 upper=0.6179939 effort=2.8 velocity=5.6548668 -> lower=-1.5708 upper=0.6179939 effort=2.8 velocity=5.6548668
- joint j_tibia_rf: limit lower=-2.6179939 upper=0.6179939 effort=2.8 velocity=5.6548668 -> lower=-1.5708 upper=0.6179939 effort=2.8 velocity=5.6548668
- joint j_tibia_rm: limit lower=-2.6179939 upper=0.6179939 effort=2.8 velocity=5.6548668 -> lower=-1.5708 upper=0.6179939 effort=2.8 velocity=5.6548668
- joint j_tibia_rr: limit lower=-2.6179939 upper=0.6179939 effort=2.8 velocity=5.6548668 -> lower=-1.5708 upper=0.6179939 effort=2.8 velocity=5.6548668

File: urdf/phantomx_urdf.xacro (robot description, xacro)
@@ -146,5 +146,5 @@
     <origin xyz="${xyz}" rpy="${rpy}" />
     <axis xyz="1 0 0" />
-    <limit effort="2.8" velocity="5.6548668" lower="-2.5179939" upper="2.5179939" />
+    <limit effort="2.8" velocity="5.6548668" lower="-0.523599" upper="0.523599" />
   </joint>
   <joint name="j_c2_${suffix}" type="fixed">
@@ -158,5 +158,5 @@
     <origin xyz="0 0 0" rpy=" 0 3.14159 3.14159" />
     <axis xyz="1 0 0" />
-    <limit effort="2.8" velocity="5.6548668" lower="-2.5179939" upper="2.5179939" />
+    <limit effort="2.8" velocity="5.6548668" lower="-1.5708" upper="1.5708" />
   </joint>
   <joint name="j_tibia_${suffix}" type="revolute">
@@ -165,5 +165,5 @@
     <origin xyz="0 ${thigh_offset_y} ${thigh_offset_z}" rpy="-1.5707 0 3.14159" />
     <axis xyz="1 0 0" />
-    <limit effort="2.8" velocity="5.6548668" lower="-2.6179939" upper="0.6179939" />
+    <limit effort="2.8" velocity="5.6548668" lower="-1.5708" upper="0.6179939" />
   </joint>
    <transmission name="t_c1_${suffix}">

Commit message: use more realistic weights and adjust color

File: urdf/phantomx.urdf (robot description, URDF)
Before this commit: robot PhantomX, 26 links, 25 joints
Links:
- link MP_BODY: mass 1.97559947 -> 1.4
- link c1_lf: mass 0.324357719 -> 0.015
- link c1_lm: mass 0.324357719 -> 0.015
- link c1_lr: mass 0.324357719 -> 0.015
- link c1_rf: mass 0.324357719 -> 0.015
- link c1_rm: mass 0.324357719 -> 0.015
- link c1_rr: mass 0.324357719 -> 0.015
- link c2_lf: mass 0.324357719 -> 0.015
- link c2_lm: mass 0.324357719 -> 0.015
- link c2_lr: mass 0.324357719 -> 0.015
- link c2_rf: mass 0.324357719 -> 0.015
- link c2_rm: mass 0.324357719 -> 0.015
- link c2_rr: mass 0.324357719 -> 0.015
- link thigh_lf: mass 0.324357719 -> 0.07
- link thigh_lm: mass 0.324357719 -> 0.07
- link thigh_lr: mass 0.324357719 -> 0.07
- link thigh_rf: mass 0.324357719 -> 0.07
- link thigh_rm: mass 0.324357719 -> 0.07
- link thigh_rr: mass 0.324357719 -> 0.07
- link tibia_lf: mass 0.324357719 -> 0.08
- link tibia_lm: mass 0.324357719 -> 0.08
- link tibia_lr: mass 0.324357719 -> 0.08
- link tibia_rf: mass 0.324357719 -> 0.08
- link tibia_rm: mass 0.324357719 -> 0.08
- link tibia_rr: mass 0.324357719 -> 0.08
Joints:
- joint j_c1_lf: limit lower=-0.523599 upper=0.523599 effort=2.8 velocity=5.6548668 -> lower=-1.0 upper=1.0 effort=2.8 velocity=5.6548668
- joint j_c1_lm: limit lower=-0.523599 upper=0.523599 effort=2.8 velocity=5.6548668 -> lower=-1.0 upper=1.0 effort=2.8 velocity=5.6548668
- joint j_c1_lr: limit lower=-0.523599 upper=0.523599 effort=2.8 velocity=5.6548668 -> lower=-1.0 upper=1.0 effort=2.8 velocity=5.6548668
- joint j_c1_rf: limit lower=-0.523599 upper=0.523599 effort=2.8 velocity=5.6548668 -> lower=-1.0 upper=1.0 effort=2.8 velocity=5.6548668
- joint j_c1_rm: limit lower=-0.523599 upper=0.523599 effort=2.8 velocity=5.6548668 -> lower=-1.0 upper=1.0 effort=2.8 velocity=5.6548668
- joint j_c1_rr: limit lower=-0.523599 upper=0.523599 effort=2.8 velocity=5.6548668 -> lower=-1.0 upper=1.0 effort=2.8 velocity=5.6548668
- joint j_thigh_lf: limit lower=-1.5708 upper=1.5708 effort=2.8 velocity=5.6548668 -> lower=-2.25 upper=2.25 effort=2.8 velocity=5.6548668
- joint j_thigh_lm: limit lower=-1.5708 upper=1.5708 effort=2.8 velocity=5.6548668 -> lower=-2.25 upper=2.25 effort=2.8 velocity=5.6548668
- joint j_thigh_lr: limit lower=-1.5708 upper=1.5708 effort=2.8 velocity=5.6548668 -> lower=-2.25 upper=2.25 effort=2.8 velocity=5.6548668
- joint j_thigh_rf: limit lower=-1.5708 upper=1.5708 effort=2.8 velocity=5.6548668 -> lower=-2.25 upper=2.25 effort=2.8 velocity=5.6548668
- joint j_thigh_rm: limit lower=-1.5708 upper=1.5708 effort=2.8 velocity=5.6548668 -> lower=-2.25 upper=2.25 effort=2.8 velocity=5.6548668
- joint j_thigh_rr: limit lower=-1.5708 upper=1.5708 effort=2.8 velocity=5.6548668 -> lower=-2.25 upper=2.25 effort=2.8 velocity=5.6548668
- joint j_tibia_lf: limit lower=-1.5708 upper=0.6179939 effort=2.8 velocity=5.6548668 -> lower=-2.75 upper=1.0 effort=2.8 velocity=5.6548668
- joint j_tibia_lm: limit lower=-1.5708 upper=0.6179939 effort=2.8 velocity=5.6548668 -> lower=-2.75 upper=1.0 effort=2.8 velocity=5.6548668
- joint j_tibia_lr: limit lower=-1.5708 upper=0.6179939 effort=2.8 velocity=5.6548668 -> lower=-2.75 upper=1.0 effort=2.8 velocity=5.6548668
- joint j_tibia_rf: limit lower=-1.5708 upper=0.6179939 effort=2.8 velocity=5.6548668 -> lower=-2.75 upper=1.0 effort=2.8 velocity=5.6548668
- joint j_tibia_rm: limit lower=-1.5708 upper=0.6179939 effort=2.8 velocity=5.6548668 -> lower=-2.75 upper=1.0 effort=2.8 velocity=5.6548668
- joint j_tibia_rr: limit lower=-1.5708 upper=0.6179939 effort=2.8 velocity=5.6548668 -> lower=-2.75 upper=1.0 effort=2.8 velocity=5.6548668

File: urdf/phantomx_urdf.xacro (robot description, xacro)
@@ -16,5 +16,5 @@
         <inertial>
           <origin xyz="0 0 0" />
-          <mass value="1.97559947"/>
+          <mass value="1.4"/>
           <inertia ixx="3.1081800"  ixy="-0.25460189"  ixz="2.0318174" iyy="6.3787776" iyz="0.16417863" izz="5.3316425" />
         </inertial>
@@ -53,5 +53,5 @@
     <inertial>
       <origin xyz="0 -${connect_offset} 0" rpy="0 0 0"  />
-      <mass value="0.324357719"/>
+      <mass value="0.015"/>
      <inertia ixx="0.0051411124"  ixy="-0.00057530255"  ixz="-0.000024729049" iyy="0.0081915737" iyz="-0.000019223094" izz="0.0011379812" />
     </inertial>
@@ -76,5 +76,5 @@
     <inertial>
       <origin xyz="0 -${connect_offset} 0" rpy="0 0 0"  />
-      <mass value="0.324357719"/>
+      <mass value="0.015"/>
      <inertia ixx="0.0051411124"  ixy="-0.00057530255"  ixz="-0.000024729049" iyy="0.0081915737" iyz="-0.000019223094" izz="0.0011379812" />
     </inertial>
@@ -99,5 +99,5 @@
     <inertial>
       <origin xyz="0 0 0" rpy="0 0 0"  />
-      <mass value="0.324357719"/>
+      <mass value="0.07"/>
      <inertia ixx="0.0051411124"  ixy="-0.00057530255"  ixz="-0.000024729049" iyy="0.0081915737" iyz="-0.000019223094" izz="0.0011379812" />
     </inertial>
@@ -122,5 +122,5 @@
     <inertial>
       <origin xyz="0 0 0" rpy="-5 0 0"  />
-      <mass value="0.324357719"/>
+      <mass value="0.08"/>
      <inertia ixx="0.0051411124"  ixy="-0.00057530255"  ixz="-0.000024729049" iyy="0.0081915737" iyz="-0.000019223094" izz="0.0011379812" />
     </inertial>
@@ -146,5 +146,5 @@
     <origin xyz="${xyz}" rpy="${rpy}" />
     <axis xyz="1 0 0" />
-    <limit effort="2.8" velocity="5.6548668" lower="-0.523599" upper="0.523599" />
+    <limit effort="2.8" velocity="5.6548668" lower="-1.0" upper="1.0" />
   </joint>
   <joint name="j_c2_${suffix}" type="fixed">
@@ -158,5 +158,5 @@
     <origin xyz="0 0 0" rpy=" 0 3.14159 3.14159" />
     <axis xyz="1 0 0" />
-    <limit effort="2.8" velocity="5.6548668" lower="-1.5708" upper="1.5708" />
+    <limit effort="2.8" velocity="5.6548668" lower="-2.25" upper="2.25" />
   </joint>
   <joint name="j_tibia_${suffix}" type="revolute">
@@ -165,5 +165,5 @@
     <origin xyz="0 ${thigh_offset_y} ${thigh_offset_z}" rpy="-1.5707 0 3.14159" />
     <axis xyz="1 0 0" />
-    <limit effort="2.8" velocity="5.6548668" lower="-1.5708" upper="0.6179939" />
+    <limit effort="2.8" velocity="5.6548668" lower="-2.75" upper="1.0" />
   </joint>
    <transmission name="t_c1_${suffix}">
